File: woagboard.kicad_sch (KiCad schematic)
At the start: 54 parts, among them J1 TYPE-C-31-M-14, J2 UART, J3 TC2030, SW1 SW_Push_45deg, SW10 SW_Push_45deg, SW11 SW_Push_45deg, SW12 SW_Push_45deg, SW13 SW_Push_45deg, SW14 SW_Push_45deg, SW15 SW_Push_45deg, SW16 SW_Push_45deg, SW17 SW_Push_45deg, SW18 SW_Push_45deg, SW2 SW_Push_45deg, SW3 SW_Push_45deg, SW4 SW_Push_45deg, SW5 SW_Push_45deg, SW6 SW_Push_45deg, SW7 SW_Push_45deg, SW8 SW_Push_45deg, SW9 SW_Push_45deg, U1 E73-2G4M08S1C, U2 BQ24075RGT, U3 USBLC6-2, Y1 32.768kHz

Commit message: feat: initial pcb
Parts:
- removed J1: TYPE-C-31-M-14, symbol Connector:USB_C_Receptacle_USB2.0_14P
- removed J2: UART, symbol Connector_Generic:Conn_01x05
- added J1: TYPE-C-31-M-12, PCM_marbastlib-various:USB_C_Receptacle_HRO_TYPE-C-31-M-12, symbol Connector:USB_C_Receptacle_USB2.0_16P
- added J2: SWD, Connector_PinHeader_2.54mm:PinHeader_1x06_P2.54mm_Horizontal, symbol Connector_Generic:Conn_01x06
- C1, C2, C5, C7, C8: footprint (none) -> Capacitor_SMD:C_0402_1005Metric_Pad0.74x0.62mm_HandSolder
- L2: footprint (none) -> Inductor_SMD:L_0805_2012Metric_Pad1.15x1.40mm_HandSolder
- PWR1, RST1: footprint (none) -> Woagboard_Footprints:EVQ-P7C01P
- SW1, SW10, SW11, SW12, SW13, SW14, SW15, SW16, SW17, SW18, SW2, SW3, SW4, SW5, SW6, SW7, SW8, SW9: footprint (none) -> Woagboard_Footprints:Choc-V1-HS-Reversible
- TH1: footprint TestPoint:TestPoint_2Pads_Pitch5.08mm_Drill1.3mm -> TestPoint:TestPoint_2Pads_Pitch2.54mm_Drill0.8mm
- Y1: footprint (none) -> Woagboard_Footprints:Q13FC13500004
Connections:
- net +3V3: now also J2.4 (Pin_4)
- net GND: now also J1.A1 (GND), J1.A12 (GND), J1.B1 (GND), J1.B12 (GND), J2.1 (Pin_1)
- net POWER: now also U1.17 (P1.09)
- net RESET: now also J2.6 (Pin_6)
- net SWDCLK: now also J2.3 (Pin_3)
- net SWDIO: now also J2.2 (Pin_2)
- net Switch1: now also U1.3 (P0.03/AIN1)
- net Switch10: now also U1.16 (P0.08)
- net Switch11: now also U1.1 (P1.11)
- net Switch12: now also U1.40 (P1.04)
- net Switch13: now also U1.38 (P1.02)
- net Switch14: now also U1.35 (P0.24)
- net Switch15: now also U1.34 (P0.22)
- net Switch16: now also U1.41 (P0.09/NFC1)
- net Switch17: now also U1.42 (P1.06)
- net Switch18: now also U1.43 (P0.10/NFC2)
- net Switch2: now also U1.33 (P0.13)
- net Switch3: now also U1.32 (P0.20)
- net Switch4: now also U1.22 (P0.07)
- net Switch5: now also U1.18 (P0.04/AIN2)
- net Switch6: now also U1.2 (P1.10)
- net Switch7: now also U1.4 (P0.28/AIN4)
- net Switch8: now also U1.30 (P0.17)
- net Switch9: now also U1.20 (P0.12)
- net USB-D+: now also U3.4 (I/O2); no longer U3.6 (I/O1)
- net USB-D-: now also U3.6 (I/O1); no longer U3.4 (I/O2)
- net USB-Din+: now also U3.3 (I/O2), J1.A6 (D+), J1.B6 (D+); no longer U3.1 (I/O1)
- net USB-Din-: now also U3.1 (I/O1), J1.A7 (D-), J1.B7 (D-); no longer U3.3 (I/O2)
- net at R1.1: now also J1.A5 (CC1)
- net LED_CHG: now reaches LED1.1 (K), R3.1
- net CHG: now reaches R3.2, U2.9 (~{CHG})
- net VBUS: now reaches L1.1
- net VBUS: now also J1.A4 (VBUS), J1.A9 (VBUS), J1.B4 (VBUS), J1.B9 (VBUS)
- net VBUS_FLT: now reaches F1.1, L1.2
- net Bypass: now reaches JP2.1 (A), R7.1
- net at R2.2: now also J1.B5 (CC2)
- net at JP1.2 (B): now also J1.S1 (SHIELD)
- net LFXO_CLK: now reaches C7.1, U1.11 (P0.00/XL1), Y1.2
- net LFXO_RET: now reaches C8.2, U1.13 (P0.01/XL2), Y1.1
- net DCCH: now reaches L2.2, U1.25 (DCCH)
- net SWO: now reaches U1.36 (P1.00)
- net SWO: now also J3.6 (SWO), J2.5 (Pin_5)
- no-connect marks 2 -> 4
Other:
- moved on the sheet: C3, C4, C7, C8, F1, LED1, R3, Y1
